Commit message: modify andbot.xacro base mass origin

File: andbot_robot/robot_description/urdf/andbot.xacro (robot description, xacro)
@@ -119,7 +119,7 @@
     <child link="xv11"/>
 <!--    plastic model     -->
-<origin xyz="-0.022 0 ${radius_wheel+0.135}" rpy="0 0 0"/>
+<!--	<origin xyz="-0.022 0 ${radius_wheel+0.135}" rpy="0 0 0"/>	-->
 <!--	metal model	-->
-<!--	<origin xyz="0.07 0 ${radius_wheel+0.135}" rpy="0 0 0"/>-->
+<origin xyz="0.07 0 ${radius_wheel+0.135}" rpy="0 0 0"/>
   </joint>
 <joint name="IMU_joint" type="fixed">
@@ -246,4 +246,210 @@
   </joint>
 -->
+  <!-- Head link -->
+  <link name="head_link">
+    <collision>
+      <origin xyz="0 0 0" rpy="0 0 0"/>
+      <geometry>
+        <mesh filename="package://andbot_robot/robot_description/mesh/head.STL"/>
+      </geometry>
+    </collision>
+    <visual>
+      <origin xyz="0 0 0" rpy="0 0 0"/>
+      <geometry>
+        <mesh filename="package://andbot_robot/robot_description/mesh/head.STL"/>
+      </geometry>
+       <material name="Blue">
+         <color rgba="0 0 1 0.5"/>
+       </material>
+    </visual>
+    <inertial>
+      <origin xyz="0 0 0.0" rpy="0 0 0"/>
+      <mass value="1.5"/>
+      <inertia ixx="0.248" ixy="0" ixz="0" iyy="0.248" iyz="0" izz="0.008"/>
+    </inertial>
+  </link>
+  <gazebo reference="head_link">
+    <material>Gazebo/Blue</material>
+  </gazebo>
+  <!-- Base link /Head Link joint -->
+  <joint name="head_joint" type="continuous">
+    <parent link="base_link"/>
+    <child link="head_link"/>
+    <origin xyz="-0.145 0 1.075" rpy="0 0 0"/>
+    <axis xyz="0 0 1"/>
+          <limit upper="1.57" lower="-1.57" velocity="10" effort="7"/>
+	  <joint_properties damping="0.0" friction="0.0"/>
+  </joint>
+  <!-- Transmission for laser joint -->
+  <transmission name="head_trans">
+    <type>transmission_interface/SimpleTransmission</type>
+    <joint name="head_joint">
+      <hardwareInterface>EffortJointInterface</hardwareInterface>
+    </joint>
+    <actuator name="headMotor">
+      <hardwareInterface>EffortJointInterface</hardwareInterface>
+      <mechanicalWhiteuction>1</mechanicalWhiteuction>
+    </actuator>
+  </transmission>
+  <!-- left_arm_link1 link -->
+  <link name="left_arm_link1">
+    <collision>
+      <origin xyz="0 0 0" rpy="-1.5707 1.5707 0"/>
+      <geometry>
+        <mesh filename="package://andbot_robot/robot_description/mesh/arm_link1.STL"/>
+      </geometry>
+    </collision>
+    <visual>
+      <origin xyz="0 0 0" rpy="-1.5707 1.5707 0"/>
+      <geometry>
+        <mesh filename="package://andbot_robot/robot_description/mesh/arm_link1.STL"/>
+      </geometry>
+       <material name="Blue">
+         <color rgba="0 0 1 0.5"/>
+       </material>
+    </visual>
+    <inertial>
+      <origin xyz="0 0 0.00" rpy="0 0 0"/>
+      <mass value="0.75"/>
+      <inertia ixx="0.148" ixy="0" ixz="0" iyy="0.148" iyz="0" izz="0.748"/>
+    </inertial>
+  </link>
+  <gazebo reference="left_arm_link1">
+    <material>Gazebo/Blue</material>
+  </gazebo>
+  <!-- Base link /left_arm_link1 Link joint -->
+  <joint name="left_arm_link1_joint" type="fixed">
+    <parent link="base_link"/>
+    <child link="left_arm_link1"/>
+    <origin xyz="-0.145 0.185 0.909" rpy="0 0 0"/>
+  </joint>
+  <!-- Left left_arm_link2 link -->
+  <link name="left_arm_link2">
+    <collision>
+      <origin xyz="0 0 0" rpy="-1.5707 1.5707 0"/>
+      <geometry>
+        <mesh filename="package://andbot_robot/robot_description/mesh/arm_link2.STL"/>
+      </geometry>
+    </collision>
+    <visual>
+      <origin xyz="0 0 0" rpy="-1.5707 1.5707 0"/>
+      <geometry>
+        <mesh filename="package://andbot_robot/robot_description/mesh/arm_link2.STL"/>
+      </geometry>
+       <material name="Blue">
+         <color rgba="0 0 1 0.5"/>
+       </material>
+    </visual>
+    <inertial>
+      <origin xyz="0 0 0.00" rpy="0 0 0"/>
+      <mass value="0.75"/>
+      <inertia ixx="0.148" ixy="0" ixz="0" iyy="0.148" iyz="0" izz="0.748"/>
+    </inertial>
+  </link>
+  <gazebo reference="left_arm_link2">
+    <material>Gazebo/Blue</material>
+  </gazebo>
+  <!-- Base link /Left_arm_link2 Link joint -->
+  <joint name="left_arm_link2_joint" type="fixed">
+    <parent link="left_arm_link1"/>
+    <child link="left_arm_link2"/>
+    <origin xyz="0 0 -0.205" rpy="0 0 0"/>
+  </joint>
+  <!-- right_arm_link1 link -->
+  <link name="right_arm_link1">
+    <collision>
+      <origin xyz="0 0 0" rpy="1.57 1.5707 0"/>
+      <geometry>
+        <mesh filename="package://andbot_robot/robot_description/mesh/arm_link1.STL"/>
+      </geometry>
+    </collision>
+    <visual>
+      <origin xyz="0 0 0" rpy="1.57 1.5707 0"/>
+      <geometry>
+        <mesh filename="package://andbot_robot/robot_description/mesh/arm_link1.STL"/>
+      </geometry>
+       <material name="Blue">
+         <color rgba="0 0 1 0.5"/>
+       </material>
+    </visual>
+    <inertial>
+      <origin xyz="0 0 0.00" rpy="0 0 0"/>
+      <mass value="0.75"/>
+      <inertia ixx="0.148" ixy="0" ixz="0" iyy="0.148" iyz="0" izz="0.748"/>
+    </inertial>
+  </link>
+  <gazebo reference="right_arm_link1">
+    <material>Gazebo/Blue</material>
+  </gazebo>
+  <!-- Base link /Right arm_link1 Link joint -->
+  <joint name="right_arm_link1_joint" type="fixed">
+    <parent link="base_link"/>
+    <child link="right_arm_link1"/>
+    <origin xyz="-0.145 -0.185 0.909" rpy="0 0 0"/>
+  </joint>
+  <!-- right_arm_link2 link -->
+  <link name="right_arm_link2">
+    <collision>
+      <origin xyz="0 0 0" rpy="-1.5707 1.5707 3.14"/>
+      <geometry>
+        <mesh filename="package://andbot_robot/robot_description/mesh/arm_link2.STL"/>
+      </geometry>
+    </collision>
+    <visual>
+      <origin xyz="0 0 0" rpy="-1.5707 1.5707 0"/>
+      <geometry>
+        <mesh filename="package://andbot_robot/robot_description/mesh/arm_link2.STL"/>
+      </geometry>
+       <material name="Blue">
+         <color rgba="0 0 1 0.5"/>
+       </material>
+    </visual>
+    <inertial>
+      <origin xyz="0 0 0.00" rpy="0 0 0"/>
+      <mass value="0.75"/>
+      <inertia ixx="0.148" ixy="0" ixz="0" iyy="0.148" iyz="0" izz="0.748"/>
+    </inertial>
+  </link>
+  <gazebo reference="right_arm_link2">
+    <material>Gazebo/Blue</material>
+  </gazebo>
+  <!-- Base link /right_arm_link2 Link joint -->
+  <joint name="right_arm_link2_joint" type="fixed">
+    <parent link="right_arm_link1"/>
+    <child link="right_arm_link2"/>
+    <origin xyz="0 0 -0.205" rpy="0 0 0"/>
+  </joint>
+  <!-- Base link / Laser link joint -->
+  <joint name="laser_joint" type="fixed">
+    <parent link="head_link"/>
+    <child link="laser"/>
+    <origin xyz="0.1 0 -0.05" rpy="0 0 0"/>
+  </joint>
+  <!-- Laser link -->
+  <link name="laser">
+    <collision>
+      <origin xyz="0 0 0" rpy="0 1.57 0"/>
+      <geometry>
+        <cylinder length="0.08" radius="0.01"/>
+      </geometry>
+    </collision>
+    <visual>
+      <origin xyz="0 0 0" rpy="0 1.57 0"/>
+      <geometry>
+        <cylinder length="0.08" radius="0.01"/>
+      </geometry>
+    </visual>
+    <inertial>
+      <mass value="0.002"/>
+      <origin xyz="0 0 0" rpy="0 0 0"/>
+      <inertia ixx="1e-6" ixy="0" ixz="0" iyy="1e-6" iyz="0" izz="0.01"/>
+    </inertial>
+  </link>
+  <gazebo reference="laser">
+    <mu1 value="5.0"/>
+    <mu2 value="5.0"/>
+    <kp value="10000000.0"/>
+    <kd value="1.0"/>
+  </gazebo>
   <!-- Left wheel link -->
   <link name="left_wheel">
@@ -348,4 +554,294 @@
     </actuator>
   </transmission>
+<!--Sonar Link -->
+  <!-- Base link / sonar1 link joint -->
+  <joint name="sonar_1_fixed" type="fixed">
+    <parent link="base_link"/>
+    <child link="sonar_1"/>
+    <origin xyz="-0.10374 0.23695 ${0.03475+0.029}"  rpy="0 0 1.5707"/>
+  </joint>
+<!--Sonar Link1-->
+  <link name="sonar_1">
+    <collision>
+      <origin xyz="0 0 0" rpy="0 0 0"/>
+      <geometry>
+        <mesh filename="package://andbot_robot/robot_description/mesh/sonar_HC_SR04.STL"/>
+      </geometry>
+    </collision>
+    <visual>
+      <origin xyz="0 0 0" rpy="0 0 0"/>
+      <geometry>
+        <mesh filename="package://andbot_robot/robot_description/mesh/sonar_HC_SR04.STL"/>
+      </geometry>
+       <material name="Yellow">
+         <color rgba=" 1 1 0 1"/>
+       </material>
+    </visual>
+    <inertial>
+      <origin xyz="0 0 0" rpy="0 0 0"/>
+      <mass value="0.1"/>
+      <inertia ixx="0.0135" ixy="0" ixz="0" iyy="0.0135" iyz="0" izz="0.025"/>
+    </inertial>
+  </link>
+  <gazebo reference="sonar_link1">
+    <mu1 value="2.0"/>
+    <mu2 value="2.0"/>
+    <kp value="10000000.0"/>
+    <kd value="1.0"/>
+    <material>Gazebo/Yellow</material>
+  </gazebo>
+<!--Sonar Link 2-->
+  <!-- Base link / sonar2 link joint -->
+  <joint name="sonar_2_fixed" type="fixed">
+    <parent link="base_link"/>
+    <child link="sonar_2"/>
+    <origin xyz="-0.15374 0.23214 ${0.03475+0.029}"  rpy="0 0 1.5707"/>
+  </joint>
+<!--Sonar Link2-->
+  <link name="sonar_2">
+    <collision>
+      <origin xyz="0 0 0" rpy="0 0 0"/>
+      <geometry>
+        <mesh filename="package://andbot_robot/robot_description/mesh/sonar_HC_SR04.STL"/>
+      </geometry>
+    </collision>
+    <visual>
+      <origin xyz="0 0 0" rpy="0 0 0"/>
+      <geometry>
+        <mesh filename="package://andbot_robot/robot_description/mesh/sonar_HC_SR04.STL"/>
+      </geometry>
+       <material name="Yellow">
+         <color rgba=" 1 1 0 1"/>
+       </material>
+    </visual>
+    <inertial>
+      <origin xyz="0 0 0" rpy="0 0 0"/>
+      <mass value="0.1"/>
+      <inertia ixx="0.0135" ixy="0" ixz="0" iyy="0.0135" iyz="0" izz="0.025"/>
+    </inertial>
+  </link>
+  <gazebo reference="sonar_link2">
+    <mu1 value="2.0"/>
+    <mu2 value="2.0"/>
+    <kp value="10000000.0"/>
+    <kd value="1.0"/>
+    <material>Gazebo/Yellow</material>
+  </gazebo>
+  <!-- Base link / sonar3 link joint -->
+  <joint name="sonar_3_fixed" type="fixed">
+    <parent link="base_link"/>
+    <child link="sonar_3"/>
+    <origin xyz="-0.20374 0.20726 ${0.03475+0.029}"  rpy="0 0 1.5707"/>
+  </joint>
+<!--Sonar Link3-->
+  <link name="sonar_3">
+    <collision>
+      <origin xyz="0 0 0" rpy="0 0 0"/>
+      <geometry>
+        <mesh filename="package://andbot_robot/robot_description/mesh/sonar_HC_SR04.STL"/>
+      </geometry>
+    </collision>
+    <visual>
+      <origin xyz="0 0 0" rpy="0 0 0"/>
+      <geometry>
+        <mesh filename="package://andbot_robot/robot_description/mesh/sonar_HC_SR04.STL"/>
+      </geometry>
+       <material name="Yellow">
+         <color rgba=" 1 1 0 1"/>
+       </material>
+    </visual>
+    <inertial>
+      <origin xyz="0 0 0" rpy="0 0 0"/>
+      <mass value="0.1"/>
+      <inertia ixx="0.0135" ixy="0" ixz="0" iyy="0.0135" iyz="0" izz="0.025"/>
+    </inertial>
+  </link>
+  <gazebo reference="sonar_link3">
+    <mu1 value="2.0"/>
+    <mu2 value="2.0"/>
+    <kp value="10000000.0"/>
+    <kd value="1.0"/>
+    <material>Gazebo/Yellow</material>
+  </gazebo>
+  <!-- Base link / sonar4 link joint -->
+  <joint name="sonar_4_fixed" type="fixed">
+    <parent link="base_link"/>
+    <child link="sonar_4"/>
+    <origin xyz="-0.25374 0.18238 ${0.03475+0.029}"  rpy="0 0 1.5707"/>
+  </joint>
+<!--Sonar Link4-->
+  <link name="sonar_4">
+    <collision>
+      <origin xyz="0 0 0" rpy="0 0 0"/>
+      <geometry>
+        <mesh filename="package://andbot_robot/robot_description/mesh/sonar_HC_SR04.STL"/>
+      </geometry>
+    </collision>
+    <visual>
+      <origin xyz="0 0 0" rpy="0 0 0"/>
+      <geometry>
+        <mesh filename="package://andbot_robot/robot_description/mesh/sonar_HC_SR04.STL"/>
+      </geometry>
+       <material name="Yellow">
+         <color rgba=" 1 1 0 1"/>
+       </material>
+    </visual>
+    <inertial>
+      <origin xyz="0 0 0" rpy="0 0 0"/>
+      <mass value="0.1"/>
+      <inertia ixx="0.0135" ixy="0" ixz="0" iyy="0.0135" iyz="0" izz="0.025"/>
+    </inertial>
+  </link>
+  <gazebo reference="sonar_link4">
+    <mu1 value="2.0"/>
+    <mu2 value="2.0"/>
+    <kp value="10000000.0"/>
+    <kd value="1.0"/>
+    <material>Gazebo/Yellow</material>
+  </gazebo>
+  <!-- Base link / sonar5 link joint -->
+  <joint name="sonar_5_fixed" type="fixed">
+    <parent link="base_link"/>
+    <child link="sonar_5"/>
+    <origin xyz="-0.25374 -0.18238 ${0.03475+0.029}"  rpy="0 0 -1.5707"/>
+  </joint>
+<!--Sonar Link5-->
+  <link name="sonar_5">
+    <collision>
+      <origin xyz="0 0 0" rpy="0 0 0"/>
+      <geometry>
+        <mesh filename="package://andbot_robot/robot_description/mesh/sonar_HC_SR04.STL"/>
+      </geometry>
+    </collision>
+    <visual>
+      <origin xyz="0 0 0" rpy="0 0 0"/>
+      <geometry>
+        <mesh filename="package://andbot_robot/robot_description/mesh/sonar_HC_SR04.STL"/>
+      </geometry>
+       <material name="Yellow">
+         <color rgba=" 1 1 0 1"/>
+       </material>
+    </visual>
+    <inertial>
+      <origin xyz="0 0 0" rpy="0 0 0"/>
+      <mass value="0.1"/>
+      <inertia ixx="0.0135" ixy="0" ixz="0" iyy="0.0135" iyz="0" izz="0.025"/>
+    </inertial>
+  </link>
+  <gazebo reference="sonar_link5">
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
Commit message: Remove laser link and plugin

File: andbot_robot/robot_description/urdf/andbot.xacro (robot description, xacro)
@@ -420,36 +420,4 @@
     <origin xyz="0 0 -0.205" rpy="0 0 0"/>
   </joint>
-  <!-- Base link / Laser link joint -->
-  <joint name="laser_joint" type="fixed">
-    <parent link="head_link"/>
-    <child link="laser"/>
-    <origin xyz="0.1 0 -0.05" rpy="0 0 0"/>
-  </joint>
-  <!-- Laser link -->
-  <link name="laser">
-    <collision>
-      <origin xyz="0 0 0" rpy="0 1.57 0"/>
-      <geometry>
-        <cylinder length="0.08" radius="0.01"/>
-      </geometry>
-    </collision>
-    <visual>
-      <origin xyz="0 0 0" rpy="0 1.57 0"/>
-      <geometry>
-        <cylinder length="0.08" radius="0.01"/>
-      </geometry>
-    </visual>
-    <inertial>
-      <mass value="0.002"/>
-      <origin xyz="0 0 0" rpy="0 0 0"/>
-      <inertia ixx="1e-6" ixy="0" ixz="0" iyy="1e-6" iyz="0" izz="0.01"/>
-    </inertial>
-  </link>
-  <gazebo reference="laser">
-    <mu1 value="5.0"/>
-    <mu2 value="5.0"/>
-    <kp value="10000000.0"/>
-    <kd value="1.0"/>
-  </gazebo>
   <!-- Left wheel link -->
   <link name="left_wheel">
@@ -865,45 +833,4 @@
       <robotBaseFrame>base_footprint</robotBaseFrame>
     </plugin>
-  </gazebo>
-<!-- Laser plugin -->
-  <gazebo reference="laser">
-    <mu1>1.0</mu1>
-    <mu2>1.0</mu2>
-    <material>Gazebo/Blue</material>
-    <sensor type="ray" name="head_hokuyo_sensor">
-      <pose>0 0 0 0 0 0</pose>
-      <visualize>true</visualize>
-      <update_rate>50</update_rate>
-      <ray>
-        <scan>
-          <horizontal>
-            <samples>2</samples>
-            <resolution>1</resolution>
-            <min_angle>-0.001</min_angle>
-            <!-- -0.0174532925 -->
-            <max_angle>0.001</max_angle>
-            <!-- 0.0174532925 -->
-          </horizontal>
-        </scan>
-        <range>
-          <min>0.10</min>
-          <max>30.0</max>
-          <resolution>0.01</resolution>
-        </range>
-        <noise>
-          <type>gaussian</type>
-          <!-- Noise parameters based on published spec for Hokuyo laser
-		       achieving "+-30mm" accuracy at range < 10m.  A mean of 0.0m and
-		       stddev of 0.01m will put 99.7% of samples within 0.03m of the true
-		       reading. -->
-          <mean>0.0</mean>
-          <stddev>0.00</stddev>
-        </noise>
-      </ray>
-      <plugin name="gazebo_ros_head_hokuyo_controller" filename="libgazebo_ros_laser.so">
-        <topicName>scan</topicName>
-        <frameName>laser</frameName>
-      </plugin>
-    </sensor>
   </gazebo>
 <!-- xv11 plugin -->

Commit message: Modify position of ASUS xtionpro in xacro file.

File: andbot_robot/robot_description/urdf/andbot.xacro (robot description, xacro)
@@ -20,5 +20,5 @@
         <parent link="base_link"/>
         <child link="camera_link"/>
-        <origin xyz="0 0 1.2" rpy="0 0 0"/>
+        <origin xyz="-0.100 0 1.2" rpy="0 0 0"/>
       </joint>
       <link name="camera_link">

Commit message: Modify xtionpro's position in the simulation model. Include andbot_teleop_key node by altering its node name as well.

File: andbot_robot/robot_description/urdf/andbot.xacro (robot description, xacro)
@@ -20,5 +20,5 @@
         <parent link="base_link"/>
         <child link="camera_link"/>
-        <origin xyz="-0.100 0 1.2" rpy="0 0 0"/>
+        <origin xyz="-0.100 0 1.3" rpy="0 0 0"/>
       </joint>
       <link name="camera_link">

Commit message: add xv11 filter

File: andbot_robot/robot_description/urdf/andbot.xacro (robot description, xacro)
@@ -20,5 +20,5 @@
         <parent link="base_link"/>
         <child link="camera_link"/>
-        <origin xyz="-0.100 0 1.3" rpy="0 0 0"/>
+        <origin xyz="-0.100 0 0.6" rpy="0 0 0"/>
       </joint>
       <link name="camera_link">

Commit message: modify

File: andbot_robot/robot_description/urdf/andbot.xacro (robot description, xacro)
@@ -17,52 +17,53 @@
   <!-- Base footprint link-->
   <link name="base_footprint"/>
-      <joint name="camera_joint" type="fixed">
-        <parent link="base_link"/>
-        <child link="camera_link"/>
-        <origin xyz="-0.100 0 0.6" rpy="0 0 0"/>
-      </joint>
-      <link name="camera_link">
-        <inertial>
-          <mass value="0.200" />
-          <origin xyz="0 0 0" rpy="0 0 0" />
-          <inertia ixx="5.8083e-4" ixy="0" ixz="0" iyy="3.0833e-5" iyz="0" izz="5.9083e-4" />
-        </inertial>
-        <visual>
-          <origin xyz="0 0 0" rpy="0 0 0" />
-          <geometry>
-            <mesh filename="package://andbot_robot/robot_description/mesh/asus_camera_simple.dae"/>
-          </geometry>
-        </visual>
-        <collision>
-          <origin xyz="0 0 0" rpy="0 0 0" />
-          <geometry>
-            <mesh filename="package://andbot_robot/robot_description/mesh/asus_camera_simple.dae"/>
-          </geometry>
-        </collision>
-      </link>
-      <joint name="camera_depth_joint" type="fixed">
-        <origin xyz="0.0 0.049 0.0" rpy="0 0 0" />
-        <parent link="camera_link" />
-        <child link="camera_depth_frame"/>
-      </joint>
-      <link name="camera_depth_frame"/>
-      <joint name="camera_depth_optical_joint" type="fixed">
-        <origin xyz="0 0 0" rpy="${-PI/2} 0.0 ${-PI/2}" />
-        <parent link="camera_depth_frame" />
-        <child link="camera_depth_optical_frame"/>
-      </joint>
-      <link name="camera_depth_optical_frame"/>
-      <joint name="camera_rgb_joint" type="fixed">
-        <origin xyz="0.0 0.022 0.0" rpy="0 0 0" />
-        <parent link="camera_link" />
-        <child link="camera_rgb_frame"/>
-      </joint>
-      <link name="camera_rgb_frame"/>
-      <joint name="camera_rgb_optical_joint" type="fixed">
-        <origin xyz="0 0 0" rpy="${-PI/2} 0.0 ${-PI/2}" />
-        <parent link="camera_rgb_frame" />
-        <child link="camera_rgb_optical_frame"/>
-      </joint>
-      <link name="camera_rgb_optical_frame"/>
+  <joint name="camera_joint" type="fixed">
+    <parent link="base_link"/>
+    <child link="camera_link"/>
+    <origin xyz="-0.100 0 0.6" rpy="0 0 0"/>
+  </joint>
+  <link name="camera_link">
+    <inertial>
+      <mass value="0.200" />
+      <origin xyz="0 0 0" rpy="0 0 0" />
+      <inertia ixx="5.8083e-4" ixy="0" ixz="0" iyy="3.0833e-5" iyz="0" izz="5.9083e-4" />
+      </inertial>
+    <visual>
+      <origin xyz="0 0 0" rpy="0 0 0" />
+      <geometry>
+        <mesh filename="package://andbot_robot/robot_description/mesh/asus_camera_simple.dae"/>
+      </geometry>
+    </visual>
+    <collision>
+      <origin xyz="0 0 0" rpy="0 0 0" />
+      <geometry>
+        <mesh filename="package://andbot_robot/robot_description/mesh/asus_camera_simple.dae"/>
+      </geometry>
+    </collision>
+  </link>
+  <joint name="camera_depth_joint" type="fixed">
+    <origin xyz="0.0 0.049 0.0" rpy="0 0 0" />
+    <parent link="camera_link" />
+    <child link="camera_depth_frame"/>
+  </joint>
+  <link name="camera_depth_frame"/>
+  <joint name="camera_depth_optical_joint" type="fixed">
+    <origin xyz="0 0 0" rpy="${-PI/2} 0.0 ${-PI/2}" />
+    <parent link="camera_depth_frame" />
+    <child link="camera_depth_optical_frame"/>
+  </joint>
+  <link name="camera_depth_optical_frame"/>
+  <joint name="camera_rgb_joint" type="fixed">
+    <origin xyz="0.0 0.022 0.0" rpy="0 0 0" />
+    <parent link="camera_link" />
+    <child link="camera_rgb_frame"/>
+  </joint>
+  <link name="camera_rgb_frame"/>
+  <joint name="camera_rgb_optical_joint" type="fixed">
+    <origin xyz="0 0 0" rpy="${-PI/2} 0.0 ${-PI/2}" />
+    <parent link="camera_rgb_frame" />
+    <child link="camera_rgb_optical_frame"/>
+  </joint>
+  <link name="camera_rgb_optical_frame"/>
+<!--
       <gazebo reference="camera_depth_frame">
         <sensor type="depth" name="camera">
@@ -90,4 +91,5 @@
         </sensor>
       </gazebo>
+-->
   <link name="xv11">
     <collision>
@@ -850,9 +852,9 @@
         <scan>
           <horizontal>
-            <samples>180</samples>
-            <resolution>1</resolution>
-            <min_angle>-1.57</min_angle>
+            <samples>360</samples>
+            <resolution>1</resolution>
+            <min_angle>0</min_angle>
             <!-- -0.0174532925 -->
-            <max_angle>1.57</max_angle>
+            <max_angle>6.28</max_angle>
             <!-- 0.0174532925 -->
           </horizontal>
@@ -874,5 +876,5 @@
       </ray>
       <plugin name="gazebo_ros_head_hokuyo_controller" filename="libgazebo_ros_laser.so">
-        <topicName>xv11_scan</topicName>
+        <topicName>scan</topicName>
         <frameName>xv11</frameName>
       </plugin>
